File: Akku_3V3_Versorgung.kicad_pcb (KiCad board)
At the start: 2 copper layers, 0 parts

Commit message: docu
Parts:
- added BT1: 18650 Li-Ion, Battery:BatteryHolder_Keystone_1042_1x18650, F.Cu at (135.0, 65.4)
- added C1: 10uF, Capacitor_SMD:C_0805_2012Metric, F.Cu at (92.7, 78.2)
- added C2: 10uF, Capacitor_SMD:C_0805_2012Metric, F.Cu at (92.7, 81.2)
- added C3: 100nF, Capacitor_SMD:C_0603_1608Metric, F.Cu at (97.0, 78.0)
- added C4: 22uF, Capacitor_SMD:C_0805_2012Metric, F.Cu at (92.7, 84.2)
- added C5: 22uF, Capacitor_SMD:C_0805_2012Metric, F.Cu at (92.7, 87.2)
- added C6: 22uF, Capacitor_SMD:C_0805_2012Metric, F.Cu at (92.7, 90.3)
- added C7: 1uF, Capacitor_SMD:C_0603_1608Metric, F.Cu at (97.0, 80.5)
- added C8: 10uF, Capacitor_SMD:C_0805_2012Metric, F.Cu at (92.7, 93.3)
- added D1: LED rot (laedt), LED_SMD:LED_0603_1608Metric, F.Cu at (127.0, 78.0)
- added D2: LED gruen (voll), LED_SMD:LED_0603_1608Metric, F.Cu at (127.0, 80.6)
- added D3: SS14, Diode_SMD:D_SMA, F.Cu at (112.2, 90.2)
- added J1: USB_5V_IN, Connector_JST:JST_PH_B2B-PH-K_1x02_P2.00mm_Vertical, F.Cu at (119.8, 87.0)
- added L1: 22uH / >=2A, Inductor_SMD:L_Bourns_SRN6045TA, F.Cu at (120.9, 80.5)
- added Q1: FS8205A, Package_SO:TSSOP-8_4.4x3mm_P0.65mm, F.Cu at (112.5, 79.0)
- added R1: 1.2k, Resistor_SMD:R_0603_1608Metric, F.Cu at (97.0, 83.0)
- added R2: 1k, Resistor_SMD:R_0603_1608Metric, F.Cu at (97.0, 85.5)
- added R3: 1k, Resistor_SMD:R_0603_1608Metric, F.Cu at (97.0, 88.0)
- added R4: 100R, Resistor_SMD:R_0603_1608Metric, F.Cu at (97.0, 90.5)
- added R5: 1k, Resistor_SMD:R_0603_1608Metric, F.Cu at (101.0, 78.0)
- added R6: 22k, Resistor_SMD:R_0603_1608Metric, F.Cu at (101.0, 80.5)
- added R7: 3.9k, Resistor_SMD:R_0603_1608Metric, F.Cu at (101.0, 83.0)
- added R8: 100k, Resistor_SMD:R_0603_1608Metric, F.Cu at (101.0, 85.5)
- added R9: 100k, Resistor_SMD:R_0603_1608Metric, F.Cu at (101.0, 88.0)
- added U1: TP4056, Package_SO:SOIC-8-1EP_3.9x4.9mm_P1.27mm_EP2.29x3mm, F.Cu at (112.3, 84.7)
- added U2: DW01A, Package_TO_SOT_SMD:SOT-23-6, F.Cu at (105.5, 79.1)
- added U3: MT3608, Package_TO_SOT_SMD:SOT-23-6, F.Cu at (105.5, 83.7)
- added U4: AP2112K-3.3, Package_TO_SOT_SMD:SOT-23-5, F.Cu at (105.5, 88.4)

Commit message: docu
Parts:
- added P1: USB_C_Plug_USB2.0, Connector_USB:USB_C_Receptacle_GCT_USB4105-xx-A_16P_TopMnt_Horizontal, F.Cu at (132.8, 90.6)
- BT1: footprint Battery:BatteryHolder_Keystone_1042_1x18650 -> PCM_yvolodym:NCR18650B
- C1, C2, C4, C5, C6, C8: footprint Capacitor_SMD:C_0805_2012Metric -> Capacitor_SMD:C_1206_3216Metric
- C3, C7: footprint Capacitor_SMD:C_0603_1608Metric -> Capacitor_SMD:C_1206_3216Metric
- J1: value USB_5V_IN -> Conn_01x03; footprint Connector_JST:JST_PH_B2B-PH-K_1x02_P2.00mm_Vertical -> Connector_JST:JST_EH_B3B-EH-A_1x03_P2.50mm_Vertical
- R1, R2, R3, R4, R5, R6, R7, R8, R9: footprint Resistor_SMD:R_0603_1608Metric -> Resistor_SMD:R_1206_3216Metric
- moved D3 32.0 mm to (143.0, 81.8)
- moved C7 30.3 mm to (118.9, 101.3)
- moved C8 28.6 mm to (118.9, 104.6)
- moved C6 27.3 mm to (118.9, 97.9)
- moved C5 27.2 mm to (118.9, 94.6)
- moved C4 27.1 mm to (118.9, 91.2)
- moved Q1 26.5 mm to (131.3, 97.7)
- moved U1 26.5 mm to (131.1, 103.3)
- moved C2 26.4 mm to (118.9, 84.5)
- moved C1 26.4 mm to (118.9, 81.2)
- moved C3 24.1 mm to (118.9, 87.9)
- moved L1 23.3 mm to (143.0, 87.8)
- moved R9 23.2 mm to (113.3, 107.6)
- moved R8 22.5 mm to (113.3, 104.3)
- moved R7 21.8 mm to (113.3, 101.0)
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Connections:
- net /CHRG renamed Net-(D1-K)
- net /GND renamed GND
- net /PROG renamed Net-(U1-PROG)
- net /STDBY renamed Net-(D2-K)
- J1 pad 1: /VBUS -> /+3V3
- R8 pad 2: Net-(J2-Pin_3) -> Net-(J1-Pin_3)
- R9 pad 1: Net-(J2-Pin_3) -> Net-(J1-Pin_3)
