File: Akku_3V3_Versorgung.kicad_pcb (KiCad board)
At the start: 2 copper layers, 29 parts, among them J1 Conn_01x03, P1 USB_C_Plug_USB2.0, Q1 FS8205A, U1 TP4056, U2 DW01A, U3 MT3608, U4 AP2112K-3.3

Commit message: Schaltplan-Korrekturen nach Datenblatt-Review
- LDO-Eingang (U4) mit Boost-Ausgang verbunden (Netz VBOOST), vorher
  ohne Verbindung
- USB-C: Buchsen-Symbol statt Stecker (passend zu Footprint USB4105),
  CC1/CC2 je 5,1k (R10/R11) nach GND, D+/D-/SBU als No-Connect
- P1/J1-Symbole in die Projektbibliothek Akku3V3 uebernommen
- Netz VBAT_SENSE benannt
- Notiztexte an Datenblaetter angeglichen (Ladestrom 0,9A bei 1,2k,
  Eingangsbereich ab 2,4V, Boost-Verhalten bei vollem Akku)
- README an Schaltplan angepasst
- Platine geleert (Neuanfang Layout)

Co-Authored-By: Claude Opus 5.5 <noreply@anthropic.com>
Parts:
- removed BT1: 18650 Li-Ion, PCM_yvolodym:NCR18650B
- removed C1, C2, C8: 10uF, Capacitor_SMD:C_1206_3216Metric
- removed C3: 100nF, Capacitor_SMD:C_1206_3216Metric
- removed C4, C5, C6: 22uF, Capacitor_SMD:C_1206_3216Metric
- removed C7: 1uF, Capacitor_SMD:C_1206_3216Metric
- removed D1: LED rot (laedt), LED_SMD:LED_0603_1608Metric
- removed D2: LED gruen (voll), LED_SMD:LED_0603_1608Metric
- removed D3: SS14, Diode_SMD:D_SMA
- removed J1: Conn_01x03, Connector_JST:JST_EH_B3B-EH-A_1x03_P2.50mm_Vertical
- removed L1: 22uH / >=2A, Inductor_SMD:L_Bourns_SRN6045TA
- removed P1: USB_C_Plug_USB2.0, Connector_USB:USB_C_Receptacle_GCT_USB4105-xx-A_16P_TopMnt_Horizontal
- removed Q1: FS8205A, Package_SO:TSSOP-8_4.4x3mm_P0.65mm
- removed R1: 1.2k, Resistor_SMD:R_1206_3216Metric
- removed R2, R3, R5: 1k, Resistor_SMD:R_1206_3216Metric
- removed R4: 100R, Resistor_SMD:R_1206_3216Metric
- removed R6: 22k, Resistor_SMD:R_1206_3216Metric
- removed R7: 3.9k, Resistor_SMD:R_1206_3216Metric
- removed R8, R9: 100k, Resistor_SMD:R_1206_3216Metric
- removed U1: TP4056, Package_SO:SOIC-8-1EP_3.9x4.9mm_P1.27mm_EP2.29x3mm
- removed U2: DW01A, Package_TO_SOT_SMD:SOT-23-6
- removed U3: MT3608, Package_TO_SOT_SMD:SOT-23-6
- removed U4: AP2112K-3.3, Package_TO_SOT_SMD:SOT-23-5
