File: Akku_3V3_Versorgung.kicad_pcb (KiCad board)
At the start: 2 copper layers, 0 parts

Commit message: shematic review
Parts:
- added BT1: 18650 Li-Ion, PCM_yvolodym:NCR18650B, B.Cu at (130.1, 65.0)
- added C1: 10uF, Capacitor_SMD:C_1206_3216Metric, F.Cu at (95.5, 54.0)
- added C2: 10uF, Capacitor_SMD:C_1206_3216Metric, F.Cu at (101.5, 54.0)
- added C3: 100nF, Capacitor_SMD:C_1206_3216Metric, F.Cu at (112.0, 52.0)
- added C4: 22uF, Capacitor_SMD:C_1206_3216Metric, F.Cu at (101.5, 60.5)
- added C5: 22uF, Capacitor_SMD:C_1206_3216Metric, F.Cu at (120.0, 59.0)
- added C6: 22uF, Capacitor_SMD:C_1206_3216Metric, F.Cu at (98.0, 69.0)
- added C7: 1uF, Capacitor_SMD:C_1206_3216Metric, F.Cu at (120.0, 72.5)
- added C8: 10uF, Capacitor_SMD:C_1206_3216Metric, F.Cu at (127.0, 57.0)
- added D1: LED rot (laedt), LED_SMD:LED_0603_1608Metric, F.Cu at (112.0, 72.2)
- added D2: LED gruen (voll), LED_SMD:LED_0603_1608Metric, F.Cu at (112.0, 67.2)
- added D3: SS14, Diode_SMD:D_SMA, F.Cu at (119.5, 66.5)
- added J1: Conn_01x03, Connector_JST:JST_EH_B3B-EH-A_1x03_P2.50mm_Vertical, F.Cu at (137.5, 49.5)
- added L1: 22uH / >=2A, Inductor_SMD:L_Bourns_SRN6045TA, F.Cu at (135.4, 58.0)
- added P1: USB_C_Receptacle_USB2.0_16P, Connector_USB:USB_C_Receptacle_GCT_USB4105-xx-A_16P_TopMnt_Horizontal, F.Cu at (101.2, 46.1)
- added Q1: FS8205A, Package_SO:TSSOP-8_4.4x3mm_P0.65mm, F.Cu at (123.5, 49.4)
- added R1: 1.2k, Resistor_SMD:R_1206_3216Metric, F.Cu at (106.5, 57.0)
- added R10: 5.1k, Resistor_SMD:R_1206_3216Metric, F.Cu at (130.0, 44.5)
- added R11: 5.1k, Resistor_SMD:R_1206_3216Metric, F.Cu at (95.5, 60.0)
- added R2: 1k, Resistor_SMD:R_1206_3216Metric, F.Cu at (105.0, 73.5)
- added R3: 1k, Resistor_SMD:R_1206_3216Metric, F.Cu at (107.5, 62.0)
- added R4: 100R, Resistor_SMD:R_1206_3216Metric, F.Cu at (118.0, 52.0)
- added R5: 1k, Resistor_SMD:R_1206_3216Metric, F.Cu at (118.0, 46.0)
- added R6: 22k, Resistor_SMD:R_1206_3216Metric, F.Cu at (126.0, 63.5)
- added R7: 3.9k, Resistor_SMD:R_1206_3216Metric, F.Cu at (97.5, 74.0)
- added R8: 100k, Resistor_SMD:R_1206_3216Metric, F.Cu at (143.5, 44.5)
- added R9: 100k, Resistor_SMD:R_1206_3216Metric, F.Cu at (136.5, 44.5)
- added U1: TP4056, Package_SO:SOIC-8-1EP_3.9x4.9mm_P1.27mm_EP2.29x3mm, F.Cu at (104.5, 67.9)
- added U2: DW01A, Package_TO_SOT_SMD:SOT-23-6, F.Cu at (112.6, 46.0)
- added U3: MT3608, Package_TO_SOT_SMD:SOT-23-6, F.Cu at (113.4, 60.0)
- added U4: AP2112K-3.3, Package_TO_SOT_SMD:SOT-23-5, F.Cu at (130.4, 50.5)
Other:
- board outline added: 77 x 37 mm

Commit message: shematic review
Parts:
- added U5: DW01A, Package_TO_SOT_SMD:SOT-23-6, F.Cu at (151.6, 49.9)
Connections:
- C3 pad 1: Net-(U2-VCC) -> Net-(U5-VCC)
- R4 pad 2: Net-(U2-VCC) -> Net-(U5-VCC)
- R5 pad 1: Net-(U2-CS) -> Net-(U5-CS)
