File: Akku_3V3_Versorgung.kicad_pcb (KiCad board)
At the start: 2 copper layers, 77 x 37 mm, 32 parts, among them J1 Conn_01x03, P1 USB_C_Receptacle_USB2.0_16P, Q1 FS8205A, U1 TP4056, U2 DW01A, U3 MT3608, U4 AP2112K-3.3, U5 DW01A

Commit message: shematic review
Connections:
- C6 pad 1: /VBOOST -> /BAT+
Changed lines of the file:
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@@
 			(layers "F.Cu" "F.Mask" "F.Paste")
 			(roundrect_rratio 0.217391)
-			(net "/VBOOST")
+			(net "/BAT+")
 			(pintype "passive")
 		)

Commit message: shematic review
Parts:
- L1: footprint Inductor_SMD:L_Bourns_SRN6045TA -> Inductor_SMD:L_1206_3216Metric
Changed lines of the file:
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@@
 		)
 	)
-	(footprint "Inductor_SMD:L_Bourns_SRN6045TA"
+	(footprint "Inductor_SMD:L_1206_3216Metric"
 		(layer "F.Cu")
 		(at 135.425 58)
-		(descr "http://www.bourns.com/docs/product-datasheets/srn6045ta.pdf")
-		(tags "Semi-shielded Power Inductor")
+		(descr "Inductor SMD 1206 (3216 Metric), square (rectangular) end terminal, IPC-7351 nominal, (Body size source: IPC-SM-782 page 80, https://www.pcb-3d.com/wordpress/wp-content/uploads/ipc-sm-782a_amendment_1_and_2.pdf)")
+		(tags "inductor")
 		(property "Reference" "L1"
-			(at 0 -4.6 0)
+			(at 0 -1.9 0)
 			(layer "F.SilkS")
 			(effects
@@
 		)
 		(property "Value" "22uH / >=2A"
-			(at 0 4.2 0)
+			(at 0 1.9 0)
 			(layer "F.Fab")
 			(effects
@@
 		(property "Datasheet" ""
 			(at 0 0 0)
-			(unlocked yes)
 			(layer "F.Fab")
 			(hide yes)
@@
 				(font
 					(size 1.27 1.27)
-					(thickness 0.15)
 				)
 			)
@@
 		(property "Description" "Isat >= 2A, z.B. SRN6045TA-220M"
 			(at 0 0 0)
-			(unlocked yes)
 			(layer "F.Fab")
 			(hide yes)
@@
 				(font
 					(size 1.27 1.27)
+				)
+			)
+		)
+		(property "KiLib_Generator" "SMD_2terminal_chip_molded"
+			(at 0 0 0)
+			(layer "F.SilkS")
+			(hide yes)
+			(effects
+				(font
+					(size 1 1)
 					(thickness 0.15)
 				)
@@
 		(duplicate_pad_numbers_are_jumpers no)
 		(fp_line
-			(start -3.1 -3.1)
-			(end -3.1 -2.65)
+			(start -0.835242 -0.91)
+			(end 0.835242 -0.91)
 			(stroke
 				(width 0.12)
@@
 		)
 		(fp_line
-			(start -3.1 -3.1)
-			(end 3.1 -3.1)
+			(start -0.835242 0.91)
+			(end 0.835242 0.91)
 			(stroke
 				(width 0.12)
@@
 			(layer "F.SilkS")
 		)
-		(fp_line
-			(start -3.1 3.1)
-			(end -3.1 2.65)
-			(stroke
-				(width 0.12)
-				(type solid)
-			)
-			(layer "F.SilkS")
-		)
-		(fp_line
-			(start 3.1 -3.1)
-			(end 3.1 -2.65)
-			(stroke
-				(width 0.12)
-				(type solid)
-			)
-			(layer "F.SilkS")
-		)
-		(fp_line
-			(start 3.1 3.1)
-			(end -3.1 3.1)
-			(stroke
-				(width 0.12)
-				(type solid)
-			)
-			(layer "F.SilkS")
-		)
-		(fp_line
-			(start 3.1 3.1)
-			(end 3.1 2.65)
-			(stroke
-				(width 0.12)
-				(type solid)
-			)
-			(layer "F.SilkS")
-		)
-		(fp_line
-			(start -3.5 -3.25)
-			(end -3.5 3.25)
+		(fp_rect
+			(start -2.35 -1.2)
+			(end 2.35 1.2)
 			(stroke
 				(width 0.05)
 				(type solid)
 			)
+			(fill no)
 			(layer "F.CrtYd")
 		)
-		(fp_line
-			(start -3.5 3.25)
-			(end 3.5 3.25)
-			(stroke
-				(width 0.05)
-				(type solid)
-			)
-			(layer "F.CrtYd")
-		)
-		(fp_line
-			(start 3.5 -3.25)
-			(end -3.5 -3.25)
-			(stroke
-				(width 0.05)
-				(type solid)
-			)
-			(layer "F.CrtYd")
-		)
-		(fp_line
-			(start 3.5 3.25)
-			(end 3.5 -3.25)
-			(stroke
-				(width 0.05)
-				(type solid)
-			)
-			(layer "F.CrtYd")
-		)
-		(fp_line
-			(start -3 -3)
-			(end -3 3)
+		(fp_rect
+			(start -1.6 -0.8)
+			(end 1.6 0.8)
 			(stroke
 				(width 0.1)
 				(type solid)
 			)
-			(layer "F.Fab")
-		)
-		(fp_line
-			(start -3 -3)
-			(end 3 -3)
-			(stroke
-				(width 0.1)
-				(type solid)
-			)
-			(layer "F.Fab")
-		)
-		(fp_line
-			(start -3 3)
-			(end 3 3)
-			(stroke
-				(width 0.1)
-				(type solid)
-			)
-			(layer "F.Fab")
-		)
-		(fp_line
-			(start 3 3)
-			(end 3 -3)
-			(stroke
-				(width 0.1)
-				(type solid)
-			)
+			(fill no)
 			(layer "F.Fab")
 		)
 		(fp_text user "${REFERENCE}"
-			(at 0 0 90)
+			(at 0 0 0)
 			(layer "F.Fab")
 			(effects
 				(font
-					(size 1 1)
-					(thickness 0.15)
+					(size 0.8 0.8)
+					(thickness 0.12)
 				)
 			)
 		)
-		(pad "1" smd rect
-			(at -2.075 0)
-			(size 2.35 5.1)
+		(pad "1" smd roundrect
+			(at -1.575 0)
+			(size 1.05 1.9)
 			(layers "F.Cu" "F.Mask" "F.Paste")
+			(roundrect_rratio 0.238095)
 			(net "/BAT+")
 			(pintype "passive")
 		)
-		(pad "2" smd rect
-			(at 2.075 0)
-			(size 2.35 5.1)
+		(pad "2" smd roundrect
+			(at 1.575 0)
+			(size 1.05 1.9)
 			(layers "F.Cu" "F.Mask" "F.Paste")
+			(roundrect_rratio 0.238095)
 			(net "/SW")
 			(pintype "passive")
 		)
 		(embedded_fonts no)
-		(model "${KICAD10_3DMODEL_DIR}/Inductor_SMD.3dshapes/L_Bourns_SRN6045TA.step"
+		(model "${KICAD10_3DMODEL_DIR}/Inductor_SMD.3dshapes/L_1206_3216Metric.step"
 			(offset
 				(xyz 0 0 0)

Commit message: shematic review
Parts:
- moved R7 32.9 mm to (130.0, 69.0), turned to -90 degrees
- moved C2 7.50 mm to (109.0, 54.0)
- moved C3 7.50 mm to (119.5, 52.0)
- moved C4 7.50 mm to (109.0, 60.5)
- moved C5 7.50 mm to (127.5, 59.0)
- moved C8 7.50 mm to (134.5, 57.0)
- moved J1 7.50 mm to (145.0, 49.5)
- moved L1 7.50 mm to (142.9, 58.0)
- moved P1 7.50 mm to (108.7, 46.1)
- moved Q1 7.50 mm to (131.0, 49.4)
- moved R1 7.50 mm to (114.0, 57.0)
- moved R10 7.50 mm to (137.5, 44.5)
- moved R3 7.50 mm to (115.0, 62.0)
- moved R4 7.50 mm to (125.5, 52.0)
- moved R5 7.50 mm to (125.5, 46.0)
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Routing:
- net GND: track 0.00 -> 205.1 mm
- net /BAT+: track 0.00 -> 156.0 mm, vias 0 -> 2
- net Net-(BT1--): track 0.00 -> 67.9 mm, vias 0 -> 2
- net Net-(U5-VCC): track 0.00 -> 55.9 mm
- net /VBUS: track 0.00 -> 50.8 mm, vias 0 -> 3
- net Net-(Q1-G1): track 0.00 -> 44.7 mm, vias 0 -> 2
- net Net-(Q1-G2): track 0.00 -> 43.6 mm, vias 0 -> 3
- net /SW: track 0.00 -> 41.1 mm, vias 0 -> 3
- net /VBOOST: track 0.00 -> 38.0 mm, vias 0 -> 3
- net Net-(U5-CS): track 0.00 -> 36.7 mm, vias 0 -> 2
- net /CC1: track 0.00 -> 29.8 mm
- net Net-(U1-PROG): track 0.00 -> 20.3 mm, vias 0 -> 2
- net /+3V3: track 0.00 -> 19.0 mm, vias 0 -> 1
- net /CC2: track 0.00 -> 16.8 mm, vias 0 -> 2
- net /VBAT_SENSE: track 0.00 -> 15.8 mm
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Other:
- board size 77 x 37 mm -> 78 x 37 mm

Commit message: shematic review
Parts:
- D1, D2: footprint LED_SMD:LED_0603_1608Metric -> LED_THT:LED_D2.0mm_W4.8mm_H2.5mm_FlatTop; moved to B.Cu
- J1, P1: moved to B.Cu
- moved D1 28.4 mm to (140.2, 75.5), turned to 180 degrees
- moved D2 22.3 mm to (132.7, 75.5), turned to 180 degrees
- moved R9 19.5 mm to (148.5, 63.5), turned to 180 degrees
- moved R8 13.6 mm to (153.0, 58.0)
- moved U5 12.3 mm to (147.1, 53.0)
- moved J1 8.50 mm to (152.5, 45.5), turned to 180 degrees
- moved U2 1.22 mm to (119.0, 45.5)
- moved P1 1.09 mm to (108.5, 45.0), turned to 0 degrees
- moved R2 0.50 mm to (105.0, 74.0)
Connections:
- BT1 pad 1: /BAT+ -> Net-(BT1-+)
Routing:
- net GND: track 205.1 -> 0.00 mm
- net /BAT+: track 156.0 -> 0.00 mm, vias 2 -> 0
- net Net-(BT1--): track 67.9 -> 0.00 mm, vias 2 -> 0
- net Net-(U5-VCC): track 55.9 -> 0.00 mm
- net /VBUS: track 50.8 -> 0.00 mm, vias 3 -> 0
- net Net-(Q1-G1): track 44.7 -> 0.00 mm, vias 2 -> 0
- net Net-(Q1-G2): track 43.6 -> 0.00 mm, vias 3 -> 0
- net /SW: track 41.1 -> 0.00 mm, vias 3 -> 0
- net /VBOOST: track 38.0 -> 0.00 mm, vias 3 -> 0
- net Net-(U5-CS): track 36.7 -> 0.00 mm, vias 2 -> 0
- net /CC1: track 29.8 -> 0.00 mm
- net Net-(U1-PROG): track 20.3 -> 0.00 mm, vias 2 -> 0
- net /+3V3: track 19.0 -> 0.00 mm, vias 1 -> 0
- net /CC2: track 16.8 -> 0.00 mm, vias 2 -> 0
- net /VBAT_SENSE: track 15.8 -> 0.00 mm
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- added copper zone on F.Cu, net GND

Commit message: shematic review
Parts:
- added SW2: SW_SPDT_XKB_DMx-xxxx-1, PCM_yvolodym:Switch_Small, B.Cu at (130.0, 45.5)
- moved U2 41.4 mm to (153.4, 68.5)
- moved R5 28.5 mm to (148.0, 63.5), turned to 0 degrees
- moved R10 22.6 mm to (158.0, 54.0)
- moved Q1 20.7 mm to (140.0, 68.0), turned to 180 degrees
- moved C7 15.0 mm to (132.0, 63.5)
- moved R9 7.54 mm to (156.0, 63.5)
- moved U3 2.08 mm to (120.5, 58.0), turned to 90 degrees
- moved D3 1.80 mm to (118.0, 67.5)
Routing:
- net /BAT+: track 0.00 -> 96.3 mm, vias 0 -> 2
- net Net-(BT1--): track 0.00 -> 87.2 mm, vias 0 -> 1
- net /VBUS: track 0.00 -> 56.2 mm, vias 0 -> 2
- net /CC1: track 0.00 -> 53.8 mm, vias 0 -> 1
- net Net-(Q1-G2): track 0.00 -> 47.5 mm
- net Net-(U5-VCC): track 0.00 -> 45.0 mm
- net /SW: track 0.00 -> 44.8 mm
- net Net-(BT1-+): track 0.00 -> 43.2 mm
- net /VBOOST: track 0.00 -> 38.1 mm, vias 0 -> 2
- net Net-(D1-K): track 0.00 -> 36.9 mm
- net /LED_R: track 0.00 -> 32.8 mm
- net Net-(D2-K): track 0.00 -> 28.8 mm
- net /+3V3: track 0.00 -> 26.6 mm, vias 0 -> 1
- net Net-(Q1-G1): track 0.00 -> 26.2 mm, vias 0 -> 2
- net /CC2: track 0.00 -> 25.1 mm, vias 0 -> 1
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